File: CAD/KiCad/DRS/HASP 2018 DRS/_saved_HASP 2018 DRS.sch (KiCad schematic (older format))
At the start: 10 parts, among them P1 CONN_02X05, U1 ATSAM3S2AA

Commit message: Add files via upload
Parts:
- gave numbers to parts that had none: 4
Changed lines of the file:
@@
 $EndComp
 $Comp
-L GND #PWR4
+L GND #PWR01
 U 1 1 5AD52460
 P 3940 4980
-F 0 "#PWR4" H 3940 4730 50  0001 C CNN
+F 0 "#PWR01" H 3940 4730 50  0001 C CNN
 F 1 "GND" H 3940 4830 50  0000 C CNN
 F 2 "" H 3940 4980 50  0000 C CNN
@@
 $EndComp
 $Comp
-L +3.3V #PWR3
+L +3.3V #PWR02
 U 1 1 5AD52517
 P 3560 2015
-F 0 "#PWR3" H 3560 1865 50  0001 C CNN
+F 0 "#PWR02" H 3560 1865 50  0001 C CNN
 F 1 "+3.3V" V 3625 2140 50  0000 C CNN
 F 2 "" H 3560 2015 50  0000 C CNN
@@
 TDI
 $Comp
-L GND #PWR5
+L GND #PWR03
 U 1 1 5AD53527
 P 5120 5160
-F 0 "#PWR5" H 5120 4910 50  0001 C CNN
+F 0 "#PWR03" H 5120 4910 50  0001 C CNN
 F 1 "GND" H 5120 5010 50  0000 C CNN
 F 2 "" H 5120 5160 50  0000 C CNN
@@
 $EndComp
 $Comp
-L GND #PWR1
+L GND #PWR04
 U 1 1 5AD53C0A
 P 2945 3565
-F 0 "#PWR1" H 2945 3315 50  0001 C CNN
+F 0 "#PWR04" H 2945 3315 50  0001 C CNN
 F 1 "GND" H 2945 3415 50  0000 C CNN
 F 2 "" H 2945 3565 50  0000 C CNN
@@
 $EndComp
 $Comp
-L GND #PWR6
+L GND #PWR05
 U 1 1 5AD53CF1
 P 5270 1710
-F 0 "#PWR6" H 5270 1460 50  0001 C CNN
+F 0 "#PWR05" H 5270 1460 50  0001 C CNN
 F 1 "GND" H 5270 1560 50  0000 C CNN
 F 2 "" H 5270 1710 50  0000 C CNN
@@
 	5870 1255 5785 1255
 $Comp
-L GND #PWR7
+L GND #PWR06
 U 1 1 5AD54271
 P 5785 955
-F 0 "#PWR7" H 5785 705 50  0001 C CNN
+F 0 "#PWR06" H 5785 705 50  0001 C CNN
 F 1 "GND" H 5785 805 50  0000 C CNN
 F 2 "" H 5785 955 50  0000 C CNN
@@
 3.3V
 $Comp
-L GND #PWR?
+L GND #PWR07
 U 1 1 5AD547E6
 P 8570 3280
-F 0 "#PWR?" H 8570 3030 50  0001 C CNN
+F 0 "#PWR07" H 8570 3030 50  0001 C CNN
 F 1 "GND" H 8570 3130 50  0000 C CNN
 F 2 "" H 8570 3280 50  0000 C CNN
@@
 $EndComp
 $Comp
-L GND #PWR?
+L GND #PWR08
 U 1 1 5AD54855
 P 8570 3380
-F 0 "#PWR?" H 8570 3130 50  0001 C CNN
+F 0 "#PWR08" H 8570 3130 50  0001 C CNN
 F 1 "GND" H 8570 3230 50  0000 C CNN
 F 2 "" H 8570 3380 50  0000 C CNN
@@
 SWDIO
 $Comp
-L GND #PWR?
+L GND #PWR09
 U 1 1 5AD549A2
 P 8570 3580
-F 0 "#PWR?" H 8570 3330 50  0001 C CNN
+F 0 "#PWR09" H 8570 3330 50  0001 C CNN
 F 1 "GND" H 8570 3430 50  0000 C CNN
 F 2 "" H 8570 3580 50  0000 C CNN
@@
 SWCLK
 $Comp
-L CONN_02X01 P?
+L CONN_02X01 P3
 U 1 1 5AD54ECD
 P 2630 2110
-F 0 "P?" H 2630 2210 50  0000 C CNN
+F 0 "P3" H 2630 2210 50  0000 C CNN
 F 1 "CONN_02X01" H 2630 2010 50  0000 C CNN
 F 2 "" H 2630 910 50  0000 C CNN
@@
 $EndComp
 $Comp
-L CONN_02X01 P?
+L CONN_02X01 P4
 U 1 1 5AD54F36
 P 2640 2405
-F 0 "P?" H 2640 2505 50  0000 C CNN
+F 0 "P4" H 2640 2505 50  0000 C CNN
 F 1 "CONN_02X01" H 2640 2305 50  0000 C CNN
 F 2 "" H 2640 1205 50  0000 C CNN
@@
 3.3V
 $Comp
-L GND #PWR?
+L GND #PWR010
 U 1 1 5AD55183
 P 2880 2110
-F 0 "#PWR?" H 2880 1860 50  0001 C CNN
+F 0 "#PWR010" H 2880 1860 50  0001 C CNN
 F 1 "GND" H 2880 1960 50  0000 C CNN
 F 2 "" H 2880 2110 50  0000 C CNN
@@
 SIGIN2
 $Comp
-L CONN_01X01 P?
+L CONN_01X01 P2
 U 1 1 5AD555CD
 P 2360 2785
-F 0 "P?" H 2360 2885 50  0000 C CNN
+F 0 "P2" H 2360 2885 50  0000 C CNN
 F 1 "CONN_01X01" V 2460 2785 50  0000 C CNN
 F 2 "" H 2360 2785 50  0000 C CNN
@@
 SIGOUT
 $Comp
-L Micro_SD_Card CON?
+L Micro_SD_Card CON1
 U 1 1 5AD5653F
 P 8980 4730
-F 0 "CON?" H 8330 5330 50  0000 C CNN
+F 0 "CON1" H 8330 5330 50  0000 C CNN
 F 1 "Micro_SD_Card" H 9630 5330 50  0000 R CNN
 F 2 "" H 10130 5030 50  0000 C CNN
@@
 $EndComp
 $Comp
-L GND #PWR?
+L GND #PWR011
 U 1 1 5AD56855
 P 8080 4530
-F 0 "#PWR?" H 8080 4280 50  0001 C CNN
+F 0 "#PWR011" H 8080 4280 50  0001 C CNN
 F 1 "GND" H 8080 4380 50  0000 C CNN
 F 2 "" H 8080 4530 50  0000 C CNN
@@
 SCK
 $Comp
-L GND #PWR?
+L GND #PWR012
 U 1 1 5AD56BED
 P 8080 4930
-F 0 "#PWR?" H 8080 4680 50  0001 C CNN
+F 0 "#PWR012" H 8080 4680 50  0001 C CNN
 F 1 "GND" H 8080 4780 50  0000 C CNN
 F 2 "" H 8080 4930 50  0000 C CNN
