File: CAD/KiCad/DRS/HASP 2018 DRS/HASP 2018 DRS.kicad_pcb (KiCad board)
At the start: 2 copper layers, 10 parts, among them CON1 Micro_SD_Card, P1 CONN_02X05, P2 CONN_01X01, P3 CONN_02X01, P4 CONN_02X01, U1 ATSAM3S2AA

Commit message: fixed rev 1 drs
Routing:
- net GND: track 22.9 -> 97.1 mm, vias 2 -> 14
- net ERASE: track 11.6 -> 9.31 mm
Other:
- board outline added: 31.5 x 20.3 mm
- rule pad_to_mask_clearance: 0.2 -> 0
