File: CAD/Eagle/Relay.brd (EAGLE design)
At the start: 42.6 x 37.1 mm, 15 parts

Commit message: gerbers
Parts:
- removed U$4: MICRO_SD, NR_connectors:MICRO_SD_HINGED
- moved JP9 66.5 mm to (59.7, 61.0)
- moved JP6 63.3 mm to (36.8, 66.0), turned to 90 degrees
- moved U$2 57.9 mm to (64.8, 20.3)
- moved JP8 50.6 mm to (52.1, 11.4)
- moved U$3 42.2 mm to (64.8, 33.0), turned to 0 degrees
- moved JP10 37.9 mm to (-7.62, 26.7)
- moved JP11 36.8 mm to (-7.62, 16.5)
- moved U$1 31.4 mm to (25.4, 40.6), turned to 270 degrees
- moved JP2 23.4 mm to (16.5, 48.3)
- moved JP3 22.0 mm to (5.08, 19.1), turned to 90 degrees
- moved JP7 17.9 mm to (14.0, 17.8), turned to 0 degrees
- moved JP4 17.7 mm to (5.08, 34.3)
- moved JP5 16.5 mm to (5.08, 26.7)
- moved JP1 9.25 mm to (5.08, 40.6), turned to 85.6 degrees
Connections:
- net SIGNAL_2 renamed SIGNAL2
- removed net PWR: U$2.1, U$3.5
- removed net SIGNAL_1: JP10.1
- removed net VDDIO: U$1.5
- new net GNDIO: U$1.P$6
- net +3V3: now also JP10.1, U$1.P$8; no longer U$1.8, U$4.VDD
- net CS: no longer U$1.12
- net DIS1: now also U$2.1
- net DIS2: now also U$3.1
- net GND: now also U$1.P$7, U$3.12; no longer U$1.6, U$1.7, U$3.8, U$4.GND1, U$4.GND2, U$4.GND3, U$4.GND4, U$4.VSS
- net INT2: now also U$3.10, U$3.3; no longer U$3.4, U$3.9
- net MISO: now also U$1.P$1; no longer U$1.1, U$4.DAT0
- net MOSI: no longer U$1.14, U$4.DAT1
- net SCK: no longer U$1.13, U$4.CLK
Routing:
- net SCK: track 29.7 -> 0.00 mm, vias 3 -> 0
- net MISO: track 25.4 -> 0.00 mm
- net MOSI: track 23.7 -> 0.00 mm, vias 2 -> 0
- net INT1: track 22.3 -> 0.00 mm
- net INT2: track 20.5 -> 0.00 mm
- net +3V3: track 14.8 -> 0.00 mm
- net RX: track 13.7 -> 0.00 mm
- net PWR: track 13.4 -> 0.00 mm, vias 2 -> 0
- net TX: track 8.05 -> 0.00 mm
- net CS: track 6.93 -> 0.00 mm
- net GND: track 1.39 -> 0.00 mm, vias 16 -> 0
- removed copper zone on layer 1, net GND
- removed copper zone on layer 16, net GND
Other:
- board size 42.6 x 37.1 mm -> 161.3 x 101.3 mm
- board text removed: "+10V"
- board text removed: "+15V"
- board text removed: "+30V"
- board text removed: "5.2018"
- board text removed: "CS"
- board text removed: "DIS1"
- board text removed: "DIS2"
- board text removed: "GND"
- board text removed: "HASP Relay Board"
- board text removed: "INT1"
- board text removed: "INT2"
- board text removed: "MISO"
- board text removed: "MOSI"
- board text removed: "RX"
- board text removed: "SCK"
- board text removed: "SIGNAL_1"
- board text removed: "SIGNAL_2"
- board text removed: "TX"
- board text removed: "V. 1"
