File: CAD/Eagle/Relay.sch (EAGLE design)
At the start: 12 parts

Commit message: gerbers
Parts:
- added U$2, U$3: (no value), relay board:EC2
Connections:
- removed net SIGNAL: JP10.1, JP11.1
- new net SIGNAL2: JP11.1
- net +3V3: now also JP10.1
- net DIS1: now also U$2.1
- net DIS2: now also U$3.1
- net GND: now also U$2.12, U$3.12
- net INT1: now also U$2.10, U$2.3
- net INT2: now also U$3.10, U$3.3
Other:
- moved on the sheet: U$1
Changed lines of the file:
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@@
 <?xml version="1.0" encoding="utf-8"?>
 <!DOCTYPE eagle SYSTEM "eagle.dtd">
-<eagle version="8.7.0">
+<eagle version="7.6.0">
 <drawing>
 <settings>
@@
 <setting verticaltext="up"/>
 </settings>
-<grid distance="0.1" unitdist="inch" unit="inch" style="lines" multiple="1" display="yes" altdistance="0.005" altunitdist="inch" altunit="inch"/>
+<grid distance="0.1" unitdist="inch" unit="inch" style="lines" multiple="1" display="no" altdistance="0.01" altunitdist="inch" altunit="inch"/>
 <layers>
 <layer number="1" name="Top" color="4" fill="1" visible="no" active="no"/>
+<layer number="2" name="Route2" color="1" fill="3" visible="no" active="no"/>
+<layer number="3" name="Route3" color="4" fill="3" visible="no" active="no"/>
+<layer number="4" name="Route4" color="1" fill="4" visible="no" active="no"/>
+<layer number="5" name="Route5" color="4" fill="4" visible="no" active="no"/>
+<layer number="6" name="Route6" color="1" fill="8" visible="no" active="no"/>
+<layer number="7" name="Route7" color="4" fill="8" visible="no" active="no"/>
+<layer number="8" name="Route8" color="1" fill="2" visible="no" active="no"/>
+<layer number="9" name="Route9" color="4" fill="2" visible="no" active="no"/>
+<layer number="10" name="Route10" color="1" fill="7" visible="no" active="no"/>
+<layer number="11" name="Route11" color="4" fill="7" visible="no" active="no"/>
+<layer number="12" name="Route12" color="1" fill="5" visible="no" active="no"/>
+<layer number="13" name="Route13" color="4" fill="5" visible="no" active="no"/>
+<layer number="14" name="Route14" color="1" fill="6" visible="no" active="no"/>
+<layer number="15" name="Route15" color="4" fill="6" visible="no" active="no"/>
 <layer number="16" name="Bottom" color="1" fill="1" visible="no" active="no"/>
 <layer number="17" name="Pads" color="2" fill="1" visible="no" active="no"/>
@@
 <part name="U$1" library="IMU" deviceset="BMI160" device=""/>
 <part name="GND1" library="supply1" deviceset="GND" device=""/>
-<part name="+3V1" library="supply1" deviceset="+3V3" device=""/>
 <part name="+3V2" library="supply1" deviceset="+3V3" device=""/>
 <part name="JP1" library="pinhead" deviceset="PINHD-1X2" device=""/>
@@
 <part name="JP10" library="pinhead" deviceset="PINHD-1X1" device=""/>
 <part name="JP11" library="pinhead" deviceset="PINHD-1X1" device=""/>
+<part name="U$2" library="relay board" deviceset="EC2" device=""/>
+<part name="U$3" library="relay board" deviceset="EC2" device=""/>
+<part name="GND3" library="supply1" deviceset="GND" device=""/>
+<part name="GND4" library="supply1" deviceset="GND" device=""/>
+<part name="+3V3" library="supply1" deviceset="+3V3" device=""/>
+<part name="+3V1" library="supply1" deviceset="+3V3" device=""/>
 </parts>
 <sheets>
@@
 <instance part="U$1" gate="G$1" x="0" y="0"/>
 <instance part="GND1" gate="1" x="0" y="-25.4"/>
-<instance part="+3V1" gate="G$1" x="-17.78" y="-25.4" rot="R90"/>
-<instance part="+3V2" gate="G$1" x="30.48" y="-20.32" rot="R180"/>
+<instance part="+3V2" gate="G$1" x="33.02" y="-12.7" rot="R270"/>
 <instance part="JP1" gate="G$1" x="-45.72" y="71.12"/>
 <instance part="JP2" gate="G$1" x="-45.72" y="55.88"/>
@@
 <instance part="JP10" gate="G$1" x="78.74" y="12.7"/>
 <instance part="JP11" gate="G$1" x="78.74" y="0"/>
+<instance part="U$2" gate="G$1" x="-111.76" y="-5.08"/>
+<instance part="U$3" gate="G$1" x="-71.12" y="-43.18"/>
+<instance part="GND3" gate="1" x="-73.66" y="-50.8"/>
+<instance part="GND4" gate="1" x="-114.3" y="-12.7"/>
+<instance part="+3V3" gate="G$1" x="66.04" y="12.7" rot="R90"/>
+<instance part="+3V1" gate="G$1" x="-17.78" y="-25.4" rot="R90"/>
 </instances>
 <busses>
@@
 <pinref part="GND2" gate="1" pin="GND"/>
 </segment>
+<segment>
+<pinref part="U$3" gate="G$1" pin="12"/>
+<wire x1="-73.66" y1="-40.64" x2="-73.66" y2="-48.26" width="0.1524" layer="91"/>
+<pinref part="GND3" gate="1" pin="GND"/>
+</segment>
+<segment>
+<pinref part="U$2" gate="G$1" pin="12"/>
+<wire x1="-114.3" y1="-2.54" x2="-114.3" y2="-10.16" width="0.1524" layer="91"/>
+<pinref part="GND4" gate="1" pin="GND"/>
+<junction x="-114.3" y="-10.16"/>
+</segment>
 </net>
 <net name="MISO" class="0">
@@
 <net name="+3V3" class="0">
 <segment>
-<wire x1="-10.16" y1="-20.32" x2="-10.16" y2="-25.4" width="0.1524" layer="91"/>
-<wire x1="-10.16" y1="-25.4" x2="-15.24" y2="-25.4" width="0.1524" layer="91"/>
-<pinref part="+3V1" gate="G$1" pin="+3V3"/>
-</segment>
-<segment>
 <pinref part="U$1" gate="G$1" pin="VDD"/>
 <wire x1="25.4" y1="-12.7" x2="30.48" y2="-12.7" width="0.1524" layer="91"/>
-<wire x1="30.48" y1="-12.7" x2="30.48" y2="-17.78" width="0.1524" layer="91"/>
 <pinref part="+3V2" gate="G$1" pin="+3V3"/>
 </segment>
+<segment>
+<pinref part="JP10" gate="G$1" pin="1"/>
+<wire x1="76.2" y1="12.7" x2="68.58" y2="12.7" width="0.1524" layer="91"/>
+<pinref part="+3V3" gate="G$1" pin="+3V3"/>
+</segment>
+<segment>
+<wire x1="-10.16" y1="-25.4" x2="-15.24" y2="-25.4" width="0.1524" layer="91"/>
+<wire x1="-10.16" y1="-20.32" x2="-10.16" y2="-25.4" width="0.1524" layer="91"/>
+<pinref part="+3V1" gate="G$1" pin="+3V3"/>
+</segment>
 </net>
 <net name="CS" class="0">
-<segment>
-<wire x1="10.16" y1="17.78" x2="10.16" y2="22.86" width="0.1524" layer="91"/>
-<label x="10.16" y="22.86" size="1.27" layer="95" rot="R90" xref="yes"/>
-</segment>
 <segment>
 <pinref part="JP6" gate="A" pin="3"/>
@@
 <net name="SCK" class="0">
 <segment>
-<wire x1="0" y1="17.78" x2="0" y2="22.86" width="0.1524" layer="91"/>
-<label x="0" y="22.86" size="1.27" layer="95" rot="R90" xref="yes"/>
-</segment>
-<segment>
 <pinref part="JP6" gate="A" pin="4"/>
 <wire x1="30.48" y1="58.42" x2="17.78" y2="58.42" width="0.1524" layer="91"/>
@@
 <net name="MOSI" class="0">
 <segment>
-<wire x1="-10.16" y1="17.78" x2="-10.16" y2="22.86" width="0.1524" layer="91"/>
-<label x="-10.16" y="22.86" size="1.27" layer="95" rot="R90" xref="yes"/>
-</segment>
-<segment>
 <pinref part="JP6" gate="A" pin="2"/>
 <wire x1="30.48" y1="63.5" x2="17.78" y2="63.5" width="0.1524" layer="91"/>
@@
 <label x="-15.24" y="71.12" size="1.27" layer="95" rot="R180" xref="yes"/>
 </segment>
+<segment>
+<pinref part="U$3" gate="G$1" pin="1"/>
+<wire x1="-73.66" y1="-15.24" x2="-73.66" y2="-7.62" width="0.1524" layer="91"/>
+<label x="-73.66" y="-7.62" size="1.778" layer="95" rot="R180" xref="yes"/>
+</segment>
 </net>
 <net name="DIS1" class="0">
@@
 <label x="-15.24" y="73.66" size="1.27" layer="95" rot="R180" xref="yes"/>
 </segment>
+<segment>
+<pinref part="U$2" gate="G$1" pin="1"/>
+<wire x1="-114.3" y1="22.86" x2="-114.3" y2="30.48" width="0.1524" layer="91"/>
+<label x="-114.3" y="30.48" size="1.778" layer="95" rot="R180" xref="yes"/>
+</segment>
 </net>
 <net name="RX" class="0">
@@
 <label x="66.04" y="38.1" size="1.27" layer="95" rot="R180" xref="yes"/>
 </segment>
+<segment>
+<pinref part="U$2" gate="G$1" pin="3"/>
+<wire x1="-106.68" y1="22.86" x2="-106.68" y2="30.48" width="0.1524" layer="91"/>
+<label x="-106.68" y="30.48" size="1.778" layer="95" rot="R90" xref="yes"/>
+</segment>
+<segment>
+<pinref part="U$2" gate="G$1" pin="10"/>
+<wire x1="-106.68" y1="-2.54" x2="-106.68" y2="-10.16" width="0.1524" layer="91"/>
+<label x="-106.68" y="-10.16" size="1.778" layer="95" rot="R270" xref="yes"/>
+</segment>
 </net>
 <net name="INT2" class="0">
@@
 <label x="66.04" y="25.4" size="1.27" layer="95" rot="R180" xref="yes"/>
 </segment>
-</net>
-<net name="SIGNAL" class="0">
-<segment>
-<pinref part="JP10" gate="G$1" pin="1"/>
-<wire x1="76.2" y1="12.7" x2="66.04" y2="12.7" width="0.1524" layer="91"/>
-<label x="66.04" y="12.7" size="1.27" layer="95" rot="R180" xref="yes"/>
-</segment>
+<segment>
+<pinref part="U$3" gate="G$1" pin="3"/>
+<wire x1="-66.04" y1="-15.24" x2="-66.04" y2="-7.62" width="0.1524" layer="91"/>
+<label x="-66.04" y="-7.62" size="1.778" layer="95" rot="R90" xref="yes"/>
+</segment>
+<segment>
+<pinref part="U$3" gate="G$1" pin="10"/>
+<wire x1="-66.04" y1="-40.64" x2="-66.04" y2="-48.26" width="0.1524" layer="91"/>
+<label x="-66.04" y="-48.26" size="1.778" layer="95" rot="R270" xref="yes"/>
+</segment>
+</net>
+<net name="SIGNAL2" class="0">
 <segment>
 <pinref part="JP11" gate="G$1" pin="1"/>
