File: Electronics/DRS SAMD21/drs.sch (EAGLE design)
At the start: 20 parts, among them U1 ATSAMD21G18

Commit message: Add files via upload
Parts:
- added JP3: (no value), pinhead:PINHD-1X1
Connections:
- new net LED: JP3.1, U1.PA27/EIC
Other:
- note added: "LED"
Changed lines of the file:
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@@
 <part name="+3V7" library="supply1" deviceset="+3V3" device=""/>
 <part name="JP2" library="pinhead" deviceset="PINHD-1X4" device=""/>
+<part name="JP3" library="pinhead" deviceset="PINHD-1X1" device=""/>
 </parts>
 <sheets>
@@
 <wire x1="144.78" y1="33.02" x2="144.78" y2="2.54" width="0.1524" layer="97" style="shortdash"/>
 <wire x1="205.74" y1="101.6" x2="205.74" y2="53.34" width="0.1524" layer="97" style="shortdash"/>
+<wire x1="175.26" y1="2.54" x2="144.78" y2="2.54" width="0.1524" layer="97" style="shortdash"/>
+<wire x1="175.26" y1="33.02" x2="175.26" y2="2.54" width="0.1524" layer="97" style="shortdash"/>
+<wire x1="160.02" y1="33.02" x2="175.26" y2="33.02" width="0.1524" layer="97" style="shortdash"/>
+<text x="152.4" y="25.4" size="5.08" layer="97">LED</text>
 </plain>
 <instances>
@@
 <instance part="+3V7" gate="G$1" x="43.18" y="15.24" rot="R90"/>
 <instance part="JP2" gate="A" x="119.38" y="15.24" rot="R180"/>
+<instance part="JP3" gate="G$1" x="152.4" y="15.24" rot="MR0"/>
 </instances>
 <busses>
@@
 </segment>
 </net>
+<net name="LED" class="0">
+<segment>
+<pinref part="JP3" gate="G$1" pin="1"/>
+<wire x1="154.94" y1="15.24" x2="162.56" y2="15.24" width="0.1524" layer="91"/>
+<label x="162.56" y="15.24" size="1.016" layer="95" xref="yes"/>
+</segment>
+<segment>
+<pinref part="U1" gate="G$1" pin="PA27/EIC"/>
+<wire x1="200.66" y1="144.78" x2="213.36" y2="144.78" width="0.1524" layer="91"/>
+<label x="213.36" y="144.78" size="1.016" layer="95" xref="yes"/>
+</segment>
+</net>
