File: Electronics/Relay Board V.2/HASP_relay_V.2.sch (EAGLE design)
At the start: 22 parts

Commit message: got rid of unnecessary things on relay board, fixed the SD card routing, set up rough pass of board size
Parts:
- removed JP4, JP7: (no value), pinhead:PINHD-1X2
- removed JP8, JP9: (no value), pinhead:PINHD-1X1
- removed R2: 47k, CRGS0603J1K5:CRGS0603J1K5
- removed U$6: CD4093BE, NAND Gates:CD4093BE
- added R3: 1M, resistor:R-US_R0603
- added R4: 47k, CRGS0603J1K5:CRGS0603J1K5
Connections:
- removed net DIS1: JP4.1
- removed net DIS2: JP4.2
- removed net N$6: U$2.5
- removed net RX: JP5.2, JP7.2
- removed net TX: JP5.1, JP7.1
- new net N$5: U$4.VSS
- net +3V3: now also R3.1, R4.1; no longer R2.2, U$6.VDD
- net COIL2: now also U$5.L; no longer U$6.J
- net CS: now also R3.2, U$4.CD
- net GND: now also U$4.CD1; no longer U$4.VSS, U$6.VSS
- net INT1: now also JP5.1; no longer JP8.1
- net INT2: now also JP5.2, R4.2, U$5.E, U$5.F; no longer JP9.1, R2.1, U$6.A, U$6.B
- net MOSI: now also U$4.CMD; no longer U$4.DAT1
- net OUT1: now also U$2.5
Other:
- moved on the sheet: JP10, JP13, JP2, JP3, JP5, JP6

Commit message: Add files via upload
Connections:
- removed net VDDIO: U$1.VDDIO
- net +3V3: now also U$1.VDDIO; no longer R1.2, R4.1, U$2.4, U$5.VDD
- net +5V: now also R1.2, R4.1, U$2.4, U$5.VDD
Changed lines of the file:
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@@
 <part name="U$1" library="IMU" deviceset="BMI160" device=""/>
 <part name="GND1" library="supply1" deviceset="GND" device=""/>
-<part name="+3V1" library="supply1" deviceset="+3V3" device=""/>
 <part name="+3V2" library="supply1" deviceset="+3V3" device=""/>
 <part name="JP1" library="pinhead" deviceset="PINHD-1X2" device=""/>
@@
 <part name="R1" library="CRGS0603J1K5" deviceset="CRGS0603J1K5" device="" value="47k"/>
 <part name="GND10" library="supply1" deviceset="GND" device=""/>
-<part name="+5V" library="supply1" deviceset="+3V3" device="" value="+5V"/>
 <part name="+3V4" library="supply1" deviceset="+3V3" device=""/>
-<part name="+5V1" library="supply1" deviceset="+3V3" device="" value="+5V"/>
-<part name="+5V3" library="supply1" deviceset="+3V3" device="" value="+5V"/>
 <part name="GND11" library="supply1" deviceset="GND" device=""/>
-<part name="+5V5" library="supply1" deviceset="+3V3" device="" value="+5V"/>
 <part name="D1" library="BAT54" deviceset="BAT54" device=""/>
 <part name="D2" library="BAT54" deviceset="BAT54" device=""/>
@@
 <part name="GND5" library="supply1" deviceset="GND" device=""/>
 <part name="R4" library="CRGS0603J1K5" deviceset="CRGS0603J1K5" device="" value="47k"/>
-<part name="+5V4" library="supply1" deviceset="+3V3" device="" value="+5V"/>
 <part name="JP5" library="pinhead" deviceset="PINHD-1X2" device=""/>
 <part name="FRAME1" library="frames" deviceset="A3L-LOC" device=""/>
+<part name="P+1" library="supply1" deviceset="+5V" device=""/>
+<part name="P+2" library="supply1" deviceset="+5V" device=""/>
+<part name="P+3" library="supply1" deviceset="+5V" device=""/>
+<part name="P+4" library="supply1" deviceset="+5V" device=""/>
+<part name="P+5" library="supply1" deviceset="+5V" device=""/>
+<part name="+3V1" library="supply1" deviceset="+3V3" device=""/>
 </parts>
 <sheets>
@@
 <instance part="U$1" gate="G$1" x="38.1" y="-15.24"/>
 <instance part="GND1" gate="1" x="38.1" y="-40.64"/>
-<instance part="+3V1" gate="G$1" x="20.32" y="-40.64" rot="R90"/>
 <instance part="+3V2" gate="G$1" x="66.04" y="-35.56" rot="R180"/>
 <instance part="JP1" gate="G$1" x="-124.46" y="68.58"/>
@@
 <instance part="R1" gate="G$1" x="-127" y="-60.96" rot="R90"/>
 <instance part="GND10" gate="1" x="-137.16" y="45.72"/>
-<instance part="+5V" gate="G$1" x="-134.62" y="73.66"/>
 <instance part="+3V4" gate="G$1" x="-137.16" y="53.34"/>
-<instance part="+5V1" gate="G$1" x="-127" y="-53.34"/>
-<instance part="+5V3" gate="G$1" x="-76.2" y="-63.5" rot="R270"/>
 <instance part="GND11" gate="1" x="-114.3" y="-99.06"/>
-<instance part="+5V5" gate="G$1" x="-129.54" y="-7.62"/>
 <instance part="D1" gate="G$1" x="-78.74" y="-7.62" rot="R90"/>
 <instance part="D2" gate="G$1" x="-38.1" y="-7.62" rot="R90"/>
@@
 <instance part="GND5" gate="1" x="12.7" y="43.18"/>
 <instance part="R4" gate="G$1" x="-66.04" y="-93.98" rot="R180"/>
-<instance part="+5V4" gate="G$1" x="-55.88" y="-93.98" rot="R270"/>
 <instance part="JP5" gate="G$1" x="-104.14" y="68.58"/>
 <instance part="FRAME1" gate="G$1" x="-170.18" y="-109.22"/>
+<instance part="P+1" gate="1" x="-134.62" y="73.66"/>
+<instance part="P+2" gate="1" x="-76.2" y="-63.5" rot="R270"/>
+<instance part="P+3" gate="1" x="-127" y="-53.34"/>
+<instance part="P+4" gate="1" x="-55.88" y="-93.98" rot="R270"/>
+<instance part="P+5" gate="1" x="-129.54" y="-7.62"/>
+<instance part="+3V1" gate="G$1" x="20.32" y="-40.64" rot="R90"/>
 </instances>
 <busses>
@@
 </segment>
 <segment>
-<pinref part="R1" gate="G$1" pin="2"/>
-<pinref part="+5V1" gate="G$1" pin="+3V3"/>
-</segment>
-<segment>
-<pinref part="+5V3" gate="G$1" pin="+3V3"/>
-<pinref part="U$5" gate="G$1" pin="VDD"/>
-<wire x1="-78.74" y1="-63.5" x2="-81.28" y2="-63.5" width="0.1524" layer="91"/>
-</segment>
-<segment>
-<pinref part="+5V5" gate="G$1" pin="+3V3"/>
-<pinref part="U$2" gate="G$1" pin="4"/>
-<wire x1="-129.54" y1="-10.16" x2="-129.54" y2="-12.7" width="0.1524" layer="91"/>
-</segment>
-<segment>
 <pinref part="R3" gate="G$1" pin="1"/>
 <wire x1="-40.64" y1="66.04" x2="-43.18" y2="66.04" width="0.1524" layer="91"/>
@@
 </segment>
 <segment>
-<pinref part="R4" gate="G$1" pin="1"/>
-<wire x1="-60.96" y1="-93.98" x2="-58.42" y2="-93.98" width="0.1524" layer="91"/>
-<pinref part="+5V4" gate="G$1" pin="+3V3"/>
+<wire x1="27.94" y1="-35.8775" x2="27.94" y2="-40.64" width="0.1524" layer="91"/>
+<wire x1="27.94" y1="-40.64" x2="22.86" y2="-40.64" width="0.1524" layer="91"/>
+<pinref part="U$1" gate="G$1" pin="VDDIO"/>
+<pinref part="+3V1" gate="G$1" pin="+3V3"/>
 </segment>
 </net>
@@
 <pinref part="JP1" gate="G$1" pin="1"/>
 <wire x1="-127" y1="71.12" x2="-134.62" y2="71.12" width="0.1524" layer="91"/>
-<pinref part="+5V" gate="G$1" pin="+3V3"/>
+<pinref part="P+1" gate="1" pin="+5V"/>
+</segment>
+<segment>
+<pinref part="U$5" gate="G$1" pin="VDD"/>
+<wire x1="-78.74" y1="-63.5" x2="-81.28" y2="-63.5" width="0.1524" layer="91"/>
+<pinref part="P+2" gate="1" pin="+5V"/>
+</segment>
+<segment>
+<pinref part="R1" gate="G$1" pin="2"/>
+<pinref part="P+3" gate="1" pin="+5V"/>
+</segment>
+<segment>
+<pinref part="R4" gate="G$1" pin="1"/>
+<wire x1="-60.96" y1="-93.98" x2="-58.42" y2="-93.98" width="0.1524" layer="91"/>
+<pinref part="P+4" gate="1" pin="+5V"/>
+</segment>
+<segment>
+<pinref part="U$2" gate="G$1" pin="4"/>
+<wire x1="-129.54" y1="-10.16" x2="-129.54" y2="-12.7" width="0.1524" layer="91"/>
+<pinref part="P+5" gate="1" pin="+5V"/>
 </segment>
 </net>
@@
 </segment>
 </net>
-<net name="VDDIO" class="0">
-<segment>
-<wire x1="27.94" y1="-35.8775" x2="27.94" y2="-40.64" width="0.1524" layer="91"/>
-<wire x1="27.94" y1="-40.64" x2="22.86" y2="-40.64" width="0.1524" layer="91"/>
-<pinref part="+3V1" gate="G$1" pin="+3V3"/>
-<pinref part="U$1" gate="G$1" pin="VDDIO"/>
-</segment>
-</net>
